Commit message: All legs have control and are able to calculate IK. Established tf2 listening for toe frames

File: install/robot_description/share/robot_description/robots/spotmicro.xacro (robot description, xacro)
@@ -61,6 +61,6 @@
       <axis xyz="1 0 0"/>
       <origin rpy="0 0 0" xyz="${shiftx} ${shifty} 0"/>
-      <limit effort="1000.0" lower="-2.548" upper="2.548" velocity="10.7"/>
-      <dynamics damping="0.0" friction="0.5"/>
+      <limit effort="10.0" lower="-2.548" upper="2.548" velocity="10.7"/>
+      <dynamics damping="1.0" friction="0.5"/>
     </joint>
   </xacro:macro>
@@ -126,6 +126,6 @@
       <axis xyz="0 1 0"/>
       <origin rpy="0 0 0" xyz="0 ${shift} 0"/>
-      <limit effort="1000.0" lower="-2.666" upper="1.548" velocity="10.5"/>
-      <dynamics damping="0.0" friction="0.0"/>
+      <limit effort="10.0" lower="-2.666" upper="1.548" velocity="10.5"/>
+      <dynamics damping="1.0" friction="0.0"/>
     </joint>
     <joint name="${pos}_leg_cover_joint" type="fixed">
@@ -172,6 +172,6 @@
       <axis xyz="0 1 0"/>
       <origin rpy="0 0 0" xyz="-0.01 0 -${leg_length}"/>
-      <limit effort="1000.0" lower="-0.1" upper="2.59" velocity="10.5"/>
-      <dynamics damping="0.0" friction="0.5"/>
+      <limit effort="10.0" lower="-0.1" upper="2.59" velocity="10.5"/>
+      <dynamics damping="1.0" friction="0.5"/>
     </joint>
   </xacro:macro>
@@ -236,5 +236,5 @@
     <inertial>
       <mass value="2.80"/>
-      <inertia ixx="0.05" ixy="0" ixz="0" iyy="0.05" iyz="0" izz="0.05" />
+      <inertia ixx="0.1" ixy="0" ixz="0" iyy="0.1" iyz="0" izz="0.1" />
     </inertial>
   </link>

Commit message: Added new URDF to improve physics (HELPED A LOT). This also probably has the last minute trajectory generator that needs to be improved

File: install/robot_description/share/robot_description/robots/spotmicro.xacro (robot description, xacro)
@@ -51,5 +51,5 @@
       <inertial>
         <mass value="0.10"/>
-        <inertia ixx="0.05" ixy="0" ixz="0" iyy="0.05" iyz="0" izz="0.05" />
+        <inertia ixx="0.01" ixy="0" ixz="0" iyy="0.01" iyz="0" izz="0.01" />
       </inertial>
     </link>
@@ -99,9 +99,4 @@
         <origin rpy="0 0 0" xyz="-0.125 -0.15 -0.02"/>
         </xacro:unless>
-<!--        <geometry>
-          <box size="0.028 0.036 ${leg_length}"/>
-        </geometry>
-        <origin rpy="0.0 0.0 0.0" xyz="0.0 0.0 -0.050"/>
-        <material name="yellow"/>-->
         <material name="black">
           <color rgba="0.0 0.0 0.0 1.0"/>
@@ -116,5 +111,5 @@
       <inertial>
         <mass value="0.15"/>
-        <inertia ixx="0.05" ixy="0" ixz="0" iyy="0.05" iyz="0" izz="0.05" />
+        <inertia ixx="0.1" ixy="0" ixz="0" iyy="0.1" iyz="0" izz="0.1" />
       </inertial>
     </link>
@@ -162,5 +157,5 @@
       <inertial>
         <mass value="0.1"/>
-        <inertia ixx="0.05" ixy="0" ixz="0" iyy="0.05" iyz="0" izz="0.05" />
+        <inertia ixx="0.1" ixy="0" ixz="0" iyy="0.1" iyz="0" izz="0.1" />
       </inertial>
     </link>
@@ -196,5 +191,5 @@
       <inertial>
         <mass value="0.05"/>
-        <inertia ixx="0.05" ixy="0" ixz="0" iyy="0.05" iyz="0" izz="0.05" />
+        <inertia ixx="0.1" ixy="0" ixz="0" iyy="0.1" iyz="0" izz="0.1" />
       </inertial>
     </link>
@@ -236,5 +231,5 @@
     <inertial>
       <mass value="2.80"/>
-      <inertia ixx="0.1" ixy="0" ixz="0" iyy="0.1" iyz="0" izz="0.1" />
+      <inertia ixx="0.01" ixy="0" ixz="0" iyy="0.01" iyz="0" izz="0.01" />
     </inertial>
   </link>
@@ -257,5 +252,5 @@
     <inertial>
       <mass value="0.20"/>
-       <inertia ixx="0.05" ixy="0" ixz="0" iyy="0.05" iyz="0" izz="0.05" />
+       <inertia ixx="0.01" ixy="0" ixz="0" iyy="0.01" iyz="0" izz="0.01" />
     </inertial>
   </link>
@@ -282,5 +277,5 @@
     <inertial>
       <mass value="0.20"/>
-      <inertia ixx="0.05" ixy="0" ixz="0" iyy="0.05" iyz="0" izz="0.05" />
+      <inertia ixx="0.01" ixy="0" ixz="0" iyy="0.01" iyz="0" izz="0.01" />
     </inertial>
   </link>

File: src/robot_description/robots/spotmicro_copy.xacro (robot description, xacro)
@@ -51,5 +51,5 @@
       <inertial>
         <mass value="0.10"/>
-        <inertia ixx="0.01" ixy="0" ixz="0" iyy="0.01" iyz="0" izz="0.01" />
+        <inertia ixx="0.05" ixy="0" ixz="0" iyy="0.05" iyz="0" izz="0.05" />
       </inertial>
     </link>
@@ -61,6 +61,6 @@
       <axis xyz="1 0 0"/>
       <origin rpy="0 0 0" xyz="${shiftx} ${shifty} 0"/>
-      <limit effort="10.0" lower="-2.548" upper="2.548" velocity="10.7"/>
-      <dynamics damping="1.0" friction="0.5"/>
+      <limit effort="1000.0" lower="-0.548" upper="0.548" velocity="0.7"/>
+      <dynamics damping="0.0" friction="0.5"/>
     </joint>
   </xacro:macro>
@@ -111,5 +111,5 @@
       <inertial>
         <mass value="0.15"/>
-        <inertia ixx="0.1" ixy="0" ixz="0" iyy="0.1" iyz="0" izz="0.1" />
+        <inertia ixx="0.05" ixy="0" ixz="0" iyy="0.05" iyz="0" izz="0.05" />
       </inertial>
     </link>
@@ -121,6 +121,6 @@
       <axis xyz="0 1 0"/>
       <origin rpy="0 0 0" xyz="0 ${shift} 0"/>
-      <limit effort="10.0" lower="-2.666" upper="1.548" velocity="10.5"/>
-      <dynamics damping="1.0" friction="0.0"/>
+      <limit effort="1000.0" lower="-2.666" upper="1.548" velocity="0.5"/>
+      <dynamics damping="0.0" friction="0.0"/>
     </joint>
     <joint name="${pos}_leg_cover_joint" type="fixed">
@@ -157,5 +157,5 @@
       <inertial>
         <mass value="0.1"/>
-        <inertia ixx="0.1" ixy="0" ixz="0" iyy="0.1" iyz="0" izz="0.1" />
+        <inertia ixx="0.05" ixy="0" ixz="0" iyy="0.05" iyz="0" izz="0.05" />
       </inertial>
     </link>
@@ -167,6 +167,6 @@
       <axis xyz="0 1 0"/>
       <origin rpy="0 0 0" xyz="-0.01 0 -${leg_length}"/>
-      <limit effort="10.0" lower="-0.1" upper="2.59" velocity="10.5"/>
-      <dynamics damping="1.0" friction="0.5"/>
+      <limit effort="1000.0" lower="-0.1" upper="2.59" velocity="0.5"/>
+      <dynamics damping="0.0" friction="0.5"/>
     </joint>
   </xacro:macro>
@@ -191,5 +191,5 @@
       <inertial>
         <mass value="0.05"/>
-        <inertia ixx="0.1" ixy="0" ixz="0" iyy="0.1" iyz="0" izz="0.1" />
+        <inertia ixx="0.05" ixy="0" ixz="0" iyy="0.05" iyz="0" izz="0.05" />
       </inertial>
     </link>
@@ -231,5 +231,5 @@
     <inertial>
       <mass value="2.80"/>
-      <inertia ixx="0.01" ixy="0" ixz="0" iyy="0.01" iyz="0" izz="0.01" />
+      <inertia ixx="0.05" ixy="0" ixz="0" iyy="0.05" iyz="0" izz="0.05" />
     </inertial>
   </link>
@@ -252,5 +252,5 @@
     <inertial>
       <mass value="0.20"/>
-       <inertia ixx="0.01" ixy="0" ixz="0" iyy="0.01" iyz="0" izz="0.01" />
+       <inertia ixx="0.05" ixy="0" ixz="0" iyy="0.05" iyz="0" izz="0.05" />
     </inertial>
   </link>
@@ -277,5 +277,5 @@
     <inertial>
       <mass value="0.20"/>
-      <inertia ixx="0.01" ixy="0" ixz="0" iyy="0.01" iyz="0" izz="0.01" />
+      <inertia ixx="0.05" ixy="0" ixz="0" iyy="0.05" iyz="0" izz="0.05" />
     </inertial>
   </link>
