Commit message: Refactored leg controller nodes to be cleaner and easier to implement gait generation and stability control. Also made all legs move to startign position together once controls launchfile is ran.

File: install/robot_description/share/robot_description/gazebo/robot.gazebo.xacro (robot description, xacro)
@@ -9,4 +9,7 @@
       <plugin filename="gz-sim-sensors-system" name="gz::sim::systems::Sensors">
         <render_engine>ogre2</render_engine>
+      </plugin>
+      <plugin filename="gz-sim-imu-system"
+              name="gz::sim::systems::Imu">
       </plugin>
     </gazebo>

File: install/robot_description/share/robot_description/robots/spotmicro_copy.xacro (robot description, xacro)
@@ -61,5 +61,5 @@
       <axis xyz="1 0 0"/>
       <origin rpy="0 0 0" xyz="${shiftx} ${shifty} 0"/>
-      <limit effort="1000.0" lower="-0.548" upper="0.548" velocity="0.7"/>
+      <limit effort="1000.0" lower="-0.548" upper="0.548" velocity="100"/>
       <dynamics damping="0.0" friction="0.5"/>
     </joint>
@@ -121,5 +121,5 @@
       <axis xyz="0 1 0"/>
       <origin rpy="0 0 0" xyz="0 ${shift} 0"/>
-      <limit effort="1000.0" lower="-2.666" upper="1.548" velocity="0.5"/>
+      <limit effort="1000.0" lower="-2.666" upper="1.548" velocity="100"/>
       <dynamics damping="0.0" friction="0.0"/>
     </joint>
@@ -167,5 +167,5 @@
       <axis xyz="0 1 0"/>
       <origin rpy="0 0 0" xyz="-0.01 0 -${leg_length}"/>
-      <limit effort="1000.0" lower="-0.1" upper="2.59" velocity="0.5"/>
+      <limit effort="1000.0" lower="-0.1" upper="2.59" velocity="100"/>
       <dynamics damping="0.0" friction="0.5"/>
     </joint>
@@ -284,4 +284,34 @@
     <child link="front_link"/>
   </joint>
+  <link name="imu_link">
+    <inertial>
+      <mass value="0.01"/>
+      <origin xyz="0 0 0" rpy="0 0 0"/>
+      <inertia ixx="0.0001" ixy="0" ixz="0" iyy="0.0001" iyz="0" izz="0.0001"/>
+    </inertial>
+  </link>
+  <joint name="imu_joint" type="fixed">
+    <parent link="base_link"/>
+    <child link="imu_link"/>
+    <origin xyz="0 0 0" rpy="0 0 0"/>
+   </joint>
+  <gazebo reference="imu_link">
+    <gravity>true</gravity>
+    <sensor name='imu_sensor' type='imu'>
+        <always_on>1</always_on>
+        <update_rate>1000</update_rate>
+        <visualize>1</visualize>
+        <topic>imu_data</topic>
+        <plugin name='imu_plugin' filename='libgazebo_ros_imu_sensor.so'>
+            <topicName>imu_data</topicName>
+            <bodyName>imu_sensor_link</bodyName>
+            <updateRateHZ>10.0</updateRateHZ>
+            <gaussianNoise>0.0</gaussianNoise>
+            <xyzOffset>0 0 0</xyzOffset>
+            <rpyOffset>0 0 0</rpyOffset>
+        </plugin>
+        <pose>0 0 0 0 0 0</pose>
+    </sensor>
+  </gazebo>
   <!-- create Legs -->
   <xacro:gen_full_leg_joint pos="front_left" shiftx="-${shiftx}" shifty="-${shifty}" shift="-${shift}" left="true"/>
