Commit message: first walking with stability attempts

File: src/robot_description/robots/spotmicro_copy.xacro (robot description, xacro)
@@ -231,5 +231,5 @@
     <inertial>
       <mass value="2.80"/>
-      <inertia ixx="0.05" ixy="0" ixz="0" iyy="0.05" iyz="0" izz="0.05" />
+      <inertia ixx="500" ixy="0" ixz="0" iyy="500" iyz="0" izz="500" />
     </inertial>
   </link>

Commit message: walking gait

File: src/robot_description/robots/spotmicro_copy.xacro (robot description, xacro)
@@ -5,4 +5,6 @@
   <xacro:property name="body_width" value="0.110" />
   <xacro:property name="body_height" value="0.070" />
+  <xacro:property name="base_mesh_path" value="file://$(find champ_description)/meshes/base_simple.stl" />
+  <xacro:property name="base_mass" value="20.0" />
   <xacro:property name="lidar_length" value="0.0985" />
   <xacro:property name="lidar_width" value="0.0577" />
@@ -61,5 +63,5 @@
       <axis xyz="1 0 0"/>
       <origin rpy="0 0 0" xyz="${shiftx} ${shifty} 0"/>
-      <limit effort="1000.0" lower="-0.548" upper="0.548" velocity="100"/>
+      <limit effort="50.0" lower="-0.548" upper="0.548" velocity="100"/>
       <dynamics damping="0.0" friction="0.5"/>
     </joint>
@@ -121,5 +123,5 @@
       <axis xyz="0 1 0"/>
       <origin rpy="0 0 0" xyz="0 ${shift} 0"/>
-      <limit effort="1000.0" lower="-2.666" upper="1.548" velocity="100"/>
+      <limit effort="50.0" lower="-2.666" upper="1.548" velocity="100"/>
       <dynamics damping="0.0" friction="0.0"/>
     </joint>
@@ -167,5 +169,5 @@
       <axis xyz="0 1 0"/>
       <origin rpy="0 0 0" xyz="-0.01 0 -${leg_length}"/>
-      <limit effort="1000.0" lower="-0.1" upper="2.59" velocity="100"/>
+      <limit effort="50.0" lower="-0.1" upper="2.59" velocity="100"/>
       <dynamics damping="0.0" friction="0.5"/>
     </joint>
@@ -230,6 +232,8 @@
     </collision>
     <inertial>
-      <mass value="2.80"/>
-      <inertia ixx="500" ixy="0" ixz="0" iyy="500" iyz="0" izz="500" />
+      <mass value="${base_mass}" />
+      <inertia ixx="${(1/12) * base_mass * (body_width * body_width + body_height * body_height)}" ixy="0.0" ixz="0.0"
+                iyy="${(1/12) * base_mass * (body_length * body_length + body_height * body_height)}" iyz="0.0"
+                izz="${(1/12) * base_mass * (body_length * body_length + body_width * body_width)}" />
     </inertial>
   </link>
